File: open_hw/smartline.kicad_pcb (KiCad board)
At the start: 2 copper layers, 40 x 20 mm, 49 parts, among them P1 USB_A_MALE, P2 CONN_01X08, P3 CONN_01X08, Q1 MMBT3904, Q2 AO3401, Q3 AO3401, U1 FT232HL, U2 93LC56B, U3 TPS73633, U4 SN74LVC1G66DRLR_SOT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

Commit message: Revert "0125_gerber_out"
This reverts commit b63fd5105e898909c3a391913cbdba684720f112.
Parts:
- added G***: LOGO, mod:liftyper_qr, B.Cu at (172.7, 96.9)

Commit message: 0125_gerber_out
Parts:
- removed G***: LOGO, mod:liftyper_qr
