File: SL_V2/sl_v2.sch (KiCad schematic (older format))
At the start: 61 parts, among them J1 USB_C_Receptacle_USB2.0, J2 Conn_02x08_Top_Bottom, Q1 AO3401A, Q2 FDC6330L, Q3 MMBT3904, U1 TPS73633DBV, U2 93LCxxB, U3 FT232H, U4 74LVC1G66, Y1 Crystal_GND24_Small

Commit message: fix sl v2 connection
Connections:
- net labels removed: 3.3V_OUT, 5V_OUT
Changed lines of the file:
@@
 7.5M_CLK
 Text Label 10250 2800 0    50   ~ 0
-3.3V_OUT
++3.3V_OUT
 Text Label 10250 2900 0    50   ~ 0
-5V_OUT
++5V_OUT
 Text Label 10250 3000 0    50   ~ 0
 GND
